File: dash_to_can/dash_to_can.kicad_sch (KiCad schematic)
At the start: 50 parts, among them J1 AVR-ISP1, J2 Conn_02x10_Top_Bottom, Q1 2N3904, Q10 AO3401A, Q2 2N3904, Q3 2N3904, Q4 AO3401A, Q5 2N3904, Q6 AO3401A, Q7 2N3904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

Commit message: updated update
Connections:
- net +12V: no longer D1.2 (A)
- net IGN: now also D1.2 (A)
Changed lines of the file:
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@@
 	(global_label "TEMP"
 		(shape input)
-		(at 149.86 154.94 0)
+		(at 149.86 154.94 180)
 		(fields_autoplaced yes)
 		(effects
@@
 				(size 1.27 1.27)
 			)
-			(justify left)
+			(justify right)
 		)
 		(property "Intersheetrefs" "${INTERSHEET_REFS}"
-			(at 157.6832 154.94 0)
+			(at 142.0368 154.94 0)
 			(effects
 				(font
 					(size 1.27 1.27)
 				)
-				(justify left)
+				(justify right)
 				(hide yes)
 			)
@@
 		)
 	)
+	(global_label "IGN"
+		(shape input)
+		(at 113.03 20.32 90)
+		(fields_autoplaced yes)
+		(effects
+			(font
+				(size 1.27 1.27)
+			)
+			(justify left)
+		)
+		(property "Intersheetrefs" "${INTERSHEET_REFS}"
+			(at 113.03 14.1295 90)
+			(effects
+				(font
+					(size 1.27 1.27)
+				)
+				(justify left)
+				(hide yes)
+			)
+		)
+	)
 	(symbol
 		(lib_id "power:+5VA")
@@
 					(unit 1)
 				)
-			)
-		)
-	)
-	(symbol
-		(lib_id "power:+12V")
-		(at 113.03 20.32 0)
-		(unit 1)
-		(exclude_from_sim no)
-		(in_bom yes)
-		(on_board yes)
-		(dnp no)
-		(fields_autoplaced yes)
-		(property "Reference" "#PWR038"
-			(at 113.03 24.13 0)
-			(effects
-				(font
-					(size 1.27 1.27)
-				)
-				(hide yes)
-			)
-		)
-		(property "Value" "+12V"
-			(at 113.03 15.24 0)
-			(effects
-				(font
-					(size 1.27 1.27)
-				)
-			)
-		)
-		(property "Footprint" ""
-			(at 113.03 20.32 0)
-			(effects
-				(font
-					(size 1.27 1.27)
-				)
-				(hide yes)
-			)
-		)
-		(property "Datasheet" ""
-			(at 113.03 20.32 0)
-			(effects
-				(font
-					(size 1.27 1.27)
-				)
-				(hide yes)
-			)
-		)
-		(property "Description" "Power symbol creates a global label with name \"+12V\""
-			(at 113.03 20.32 0)
-			(effects
-				(font
-					(size 1.27 1.27)
-				)
-				(hide yes)
-			)
-		)
-		(pin "1"
-		)
-		(instances
-			(project ""
-				(path "/700e3b52-0f03-40fd-ae99-83db74362cd5"
-					(reference "#PWR038")
-					(unit 1)
-				)

Commit message: Uploading my (Gabriel's) changes
Tweaking and organising schematic
Parts:
- added C12: 100uF, Capacitor_SMD:CP_Elec_4x3, symbol Device:C_Polarized
- added R18: 10k, Resistor_SMD:R_0201_0603Metric, symbol Device:R
- C2: value C_Polarized -> 330uF
- C3, C4: value C -> 100nF
- R10: value R -> 1K
Connections:
- net +5V: now also C7.2, R18.2; no longer C11.2, C7.1, U1.20 (AREF)
- net GND: now also C7.1, C12.2; no longer C7.2
- net at C3.1, D1.1 (K), U2.1 (VI): now also C12.1
- new net: C11.2, R18.1, U1.20 (AREF)
- no-connect marks 21 -> 20
Other:
- note added: "ATMega328P"
- note added: "Crystal Oscillator"
- note added: "Dash 20 pins"
- note added: "Indicators and Outputs"
- note added: "LM7805 5V Power Supply"
- note added: "MCP2515 CAN Controller"
- note added: "MCP41010 Digital Potentiometer"
- note added: "TJA1050T CAN Bus"
- note added: "ULN2003A High Current Driver"
- moved on the sheet: C1, C10, C11, C2, C3, C4, C7, C9, D1, D2, J1, J2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
