File: dash_to_can/dash_to_can.kicad_sch (KiCad schematic)
At the start: 60 parts, among them J1 AVR-ISP1, J2 Conn_02x10_Top_Bottom, Q1 2N3904, Q10 AO3401A, Q2 2N3904, Q3 2N3904, Q4 AO3401A, Q5 2N3904, Q6 AO3401A, Q7 2N3904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

Commit message: PCB update, still wiring to do
Parts:
- removed D3: 1N5822, Diode_THT:D_DO-201AD_P15.24mm_Horizontal, symbol Diode:1N5822
- added D1: SS32, Diode_SMD:D_SMA_Handsoldering, symbol Diode:SS32
- added H1, H2, H3, H4: MountingHole, MountingHole:MountingHole_3.2mm_M3, symbol Mechanical:MountingHole
- C1, C8: value C -> 100nF; footprint Capacitor_SMD:C_0603_1608Metric -> Capacitor_SMD:C_0805_2012Metric_Pad1.18x1.45mm_HandSolder
- C10, C11, C3, C4, C5, C6, C7, C9: footprint Capacitor_SMD:C_0603_1608Metric -> Capacitor_SMD:C_0805_2012Metric_Pad1.18x1.45mm_HandSolder
- C12, C2: footprint Capacitor_SMD:CP_Elec_4x3 -> Capacitor_THT:CP_Radial_D6.3mm_P2.50mm
- D2: footprint LED_SMD:LED_0603_1608Metric -> Diode_SMD:D_0805_2012Metric_Pad1.15x1.40mm_HandSolder
- F1: value 1k -> 12V 3A; footprint (none) -> Fuse:Fuse_0805_2012Metric_Pad1.15x1.40mm_HandSolder
- J2: footprint Connector_PinHeader_2.54mm:PinHeader_2x10_P2.54mm_Horizontal -> Connector_PinHeader_2.54mm:PinHeader_2x10_P2.54mm_Vertical
- L1: footprint (none) -> Inductor_SMD:L_TDK_SLF12575
- R1, R10, R11, R12, R13, R14, R15, R16, R18, R19, R2, R20, R21, R22, R23, R24, R3, R4, R5, R6, R7, R8, R9: footprint Resistor_SMD:R_0201_0603Metric -> Resistor_SMD:R_0805_2012Metric_Pad1.20x1.40mm_HandSolder
- R17: value 330R -> 1k; footprint Resistor_SMD:R_0201_0603Metric -> Resistor_SMD:R_0805_2012Metric_Pad1.20x1.40mm_HandSolder
- Y1, Y2: footprint Crystal:Crystal_SMD_5032-2Pin_5.0x3.2mm -> Crystal:Crystal_HC49-4H_Vertical
Connections:
- net +5V: now also D2.2 (A); no longer R17.1
- net GND: now also R17.1, D1.2 (A); no longer D2.1 (K)
- net at L1.1, U2.2 (OUT): now also D1.1 (K)
- net at R17.2: now also D2.1 (K); no longer D2.2 (A)
Other:
- note added: "LM2575 5V Power Supply"
- note removed: "LM7805 5V Power Supply"
- moved on the sheet: C1, C12, C2, C3, C4, C8, F1, J1, L1, U2
