File: dash_to_can/dash_to_can.kicad_sch (KiCad schematic)
At the start: 64 parts, among them J1 AVR-ISP1, J2 Conn_02x10_Top_Bottom, Q1 2N3904, Q10 AO3401A, Q2 2N3904, Q3 2N3904, Q4 AO3401A, Q5 2N3904, Q6 AO3401A, Q7 2N3904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

Commit message: Second Draft
Parts:
- Q1, Q2, Q3, Q5, Q7, Q9: footprint Package_TO_SOT_THT:TO-92_Inline -> Package_TO_SOT_SMD:SOT-23
Connections:
- net D1: now also U1.11 (PD7); no longer U1.9 (PD5)
- net D3: now also U1.9 (PD5); no longer U1.11 (PD7)
- net FUEL: now also J2.17 (Pin_17); no longer J2.16 (Pin_16)
- net ILLUM: now also Q4.3 (D), R21.2; no longer Q8.3 (D), R24.2
- net ILLUM DRIVER: now also Q5.2 (B), R11.2; no longer Q9.2 (B), R13.2
- net R DRIVER: now also Q9.2 (B), R13.2; no longer Q5.2 (B), R11.2
- net TEMP: now also J2.16 (Pin_16); no longer J2.17 (Pin_17)
- net TURN R: now also Q8.3 (D), R24.2; no longer Q4.3 (D), R21.2
Changed lines of the file:
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@@
 		)
 	)
-	(global_label "ILLUM DRIVER"
+	(global_label "R DRIVER"
 		(shape input)
 		(at 83.82 182.88 180)
@@
 		)
 		(property "Intersheetrefs" "${INTERSHEET_REFS}"
-			(at 67.7719 182.88 0)
+			(at 71.9448 182.88 0)
 			(effects
 				(font
@@
 		)
 	)
-	(global_label "R DRIVER"
+	(global_label "ILLUM DRIVER"
 		(shape input)
 		(at 267.97 60.96 0)
@@
 		)
 		(property "Intersheetrefs" "${INTERSHEET_REFS}"
-			(at 279.8452 60.96 0)
+			(at 284.0181 60.96 0)
 			(effects
 				(font
@@
 		)
 	)
-	(global_label "ILLUM"
+	(global_label "TURN R"
 		(shape input)
 		(at 115.57 182.88 0)
@@
 		)
 		(property "Intersheetrefs" "${INTERSHEET_REFS}"
-			(at 123.9981 182.88 0)
+			(at 125.6914 182.88 0)
 			(effects
 				(font
@@
 		)
 	)
-	(global_label "TEMP"
+	(global_label "FUEL"
 		(shape input)
 		(at 139.7 102.87 0)
@@
 		)
 		(property "Intersheetrefs" "${INTERSHEET_REFS}"
-			(at 147.5232 102.87 0)
+			(at 147.2814 102.87 0)
 			(effects
 				(font
@@
 		)
 	)
-	(global_label "D3"
+	(global_label "D1"
 		(shape input)
 		(at 267.97 99.06 0)
@@
 		)
 	)
-	(global_label "R DRIVER"
+	(global_label "ILLUM DRIVER"
 		(shape input)
 		(at 20.32 151.13 180)
@@
 		)
 		(property "Intersheetrefs" "${INTERSHEET_REFS}"
-			(at 8.4448 151.13 0)
+			(at 4.2719 151.13 0)
 			(effects
 				(font
@@
 		)
 	)
-	(global_label "TURN R"
+	(global_label "ILLUM"
 		(shape input)
 		(at 50.8 151.13 0)
@@
 		)
 	)
-	(global_label "ILLUM DRIVER"
+	(global_label "R DRIVER"
 		(shape input)
 		(at 267.97 73.66 0)
@@
 		)
 		(property "Intersheetrefs" "${INTERSHEET_REFS}"
-			(at 284.0181 73.66 0)
+			(at 279.8452 73.66 0)
 			(effects
 				(font
@@
 		)
 	)
-	(global_label "D1"
+	(global_label "D3"
 		(shape input)
 		(at 267.97 93.98 0)
@@
 		)
 	)
-	(global_label "FUEL"
+	(global_label "TEMP"
 		(shape input)
 		(at 139.7 100.33 0)
@@
 		)
 		(property "Intersheetrefs" "${INTERSHEET_REFS}"
-			(at 147.2814 100.33 0)
+			(at 147.5232 100.33 0)
 			(effects
 				(font
@@
 			)
 		)
-		(property "Footprint" "Package_TO_SOT_THT:TO-92_Inline"
+		(property "Footprint" "Package_TO_SOT_SMD:SOT-23"
 			(at 95.25 184.785 0)
 			(effects
@@
 			)
 		)
-		(property "Footprint" "Package_TO_SOT_THT:TO-92_Inline"
+		(property "Footprint" "Package_TO_SOT_SMD:SOT-23"
 			(at 153.67 153.035 0)
 			(effects
@@
 			)
 		)
-		(property "Footprint" "Package_TO_SOT_THT:TO-92_Inline"
+		(property "Footprint" "Package_TO_SOT_SMD:SOT-23"
 			(at 40.64 184.785 0)
 			(effects
@@
 			)
 		)
-		(property "Footprint" "Package_TO_SOT_THT:TO-92_Inline"
+		(property "Footprint" "Package_TO_SOT_SMD:SOT-23"
 			(at 31.75 153.035 0)
 			(effects
@@
 			)
 		)
-		(property "Footprint" "Package_TO_SOT_THT:TO-92_Inline"
+		(property "Footprint" "Package_TO_SOT_SMD:SOT-23"
 			(at 86.36 153.035 0)
 			(effects
@@
 			)
 		)
-		(property "Footprint" "Package_TO_SOT_THT:TO-92_Inline"
+		(property "Footprint" "Package_TO_SOT_SMD:SOT-23"
 			(at 153.67 183.515 0)
 			(effects
