File: dash_to_can/dash_to_can.kicad_pcb (KiCad board)
At the start: 2 copper layers, 100 x 100 mm, 50 parts, among them J1 AVR-ISP1, J2 Conn_02x10_Top_Bottom, Q1 2N3904, Q10 AO3401A, Q2 2N3904, Q3 2N3904, Q4 AO3401A, Q5 2N3904, Q6 AO3401A, Q7 2N3904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

Commit message: Uploading my (Gabriel's) changes
Tweaking and organising schematic
Parts:
- added C12: 100uF, Capacitor_SMD:CP_Elec_4x3, F.Cu at (119.3, 33.7)
- added R18: 10k, Resistor_SMD:R_0201_0603Metric, F.Cu at (116.7, 37.5)
- C2: value C_Polarized -> 330uF
- C3, C4: value C -> 100nF
- R10: value R -> 1K
Connections:
- C11 pad 2: +5V -> Net-(U1-AREF)
- C7 pad 1: +5V -> GND
- C7 pad 2: GND -> +5V
- U1 pad 20: +5V -> Net-(U1-AREF)

Commit message: PCB update, still wiring to do
Parts:
- added F1: 12V 3A, Fuse:Fuse_0805_2012Metric_Pad1.15x1.40mm_HandSolder, F.Cu at (145.0, 100.5)
- added H1: MountingHole, MountingHole:MountingHole_3.2mm_M3, F.Cu at (78.0, 32.0)
- added H2: MountingHole, MountingHole:MountingHole_3.2mm_M3, F.Cu at (170.0, 32.0)
- added H3: MountingHole, MountingHole:MountingHole_3.2mm_M3, F.Cu at (170.0, 124.0)
- added H4: MountingHole, MountingHole:MountingHole_3.2mm_M3, F.Cu at (78.0, 124.0)
- added L1: 100uH, Inductor_SMD:L_TDK_SLF12575, F.Cu at (123.5, 102.9)
- added R19: 10k, Resistor_SMD:R_0805_2012Metric_Pad1.20x1.40mm_HandSolder, B.Cu at (113.5, 78.5)
- added R20: 10k, Resistor_SMD:R_0805_2012Metric_Pad1.20x1.40mm_HandSolder, B.Cu at (108.3, 71.0)
- added R21: 100k, Resistor_SMD:R_0805_2012Metric_Pad1.20x1.40mm_HandSolder, F.Cu at (125.0, 43.2)
- added R22: 100k, Resistor_SMD:R_0805_2012Metric_Pad1.20x1.40mm_HandSolder, F.Cu at (104.0, 43.2)
- added R23: 100k, Resistor_SMD:R_0805_2012Metric_Pad1.20x1.40mm_HandSolder, F.Cu at (118.0, 43.2)
- added R24: 100k, Resistor_SMD:R_0805_2012Metric_Pad1.20x1.40mm_HandSolder, F.Cu at (111.0, 43.2)
- C1: value C -> 100nF; footprint Capacitor_SMD:C_0603_1608Metric -> Capacitor_SMD:C_0805_2012Metric_Pad1.18x1.45mm_HandSolder; moved to B.Cu
- C10, C9: value C -> 22pF; footprint Capacitor_SMD:C_0603_1608Metric -> Capacitor_SMD:C_0805_2012Metric_Pad1.18x1.45mm_HandSolder
- C11: footprint Capacitor_SMD:C_0603_1608Metric -> Capacitor_SMD:C_0805_2012Metric_Pad1.18x1.45mm_HandSolder; moved to B.Cu
- C12, C2: footprint Capacitor_SMD:CP_Elec_4x3 -> Capacitor_THT:CP_Radial_D6.3mm_P2.50mm
- C3, C4: footprint Capacitor_SMD:C_0603_1608Metric -> Capacitor_SMD:C_0805_2012Metric_Pad1.18x1.45mm_HandSolder
- C5, C6: value 22pf -> 16pF; footprint Capacitor_SMD:C_0603_1608Metric -> Capacitor_SMD:C_0805_2012Metric_Pad1.18x1.45mm_HandSolder; moved to B.Cu
- C7: footprint Capacitor_SMD:C_0603_1608Metric -> Capacitor_SMD:C_0805_2012Metric_Pad1.18x1.45mm_HandSolder; moved to F.Cu
- C8: value C -> 100nF; footprint Capacitor_SMD:C_0603_1608Metric -> Capacitor_SMD:C_0805_2012Metric_Pad1.18x1.45mm_HandSolder
- D1: value 1N4007 -> SS32; footprint Diode_THT:D_DO-41_SOD81_P10.16mm_Horizontal -> Diode_SMD:D_SMA_Handsoldering
- D2: footprint LED_SMD:LED_0603_1608Metric -> Diode_SMD:D_0805_2012Metric_Pad1.15x1.40mm_HandSolder
- J1, Q10, U4, U5, U6: moved to F.Cu
- J2: footprint Connector_PinHeader_2.54mm:PinHeader_2x10_P2.54mm_Horizontal -> Connector_PinHeader_2.54mm:PinHeader_2x10_P2.54mm_Vertical
- R1, R11, R13, R16, R18, R2, R4, R5, R7: footprint Resistor_SMD:R_0201_0603Metric -> Resistor_SMD:R_0805_2012Metric_Pad1.20x1.40mm_HandSolder; moved to B.Cu
- R10: value 1K -> 1k; footprint Resistor_SMD:R_0201_0603Metric -> Resistor_SMD:R_0805_2012Metric_Pad1.20x1.40mm_HandSolder
- R12, R14, R3, R6, R8: footprint Resistor_SMD:R_0201_0603Metric -> Resistor_SMD:R_0805_2012Metric_Pad1.20x1.40mm_HandSolder
- R15: value R -> 10M; footprint Resistor_SMD:R_0201_0603Metric -> Resistor_SMD:R_0805_2012Metric_Pad1.20x1.40mm_HandSolder
- R17: value R -> 1k; footprint Resistor_SMD:R_0201_0603Metric -> Resistor_SMD:R_0805_2012Metric_Pad1.20x1.40mm_HandSolder; moved to B.Cu
- R9: footprint Resistor_SMD:R_0201_0603Metric -> Resistor_SMD:R_0805_2012Metric_Pad1.20x1.40mm_HandSolder; moved to F.Cu
- U2: value LM7805_TO220 -> LM2575-5.0BU; footprint Package_TO_SOT_THT:TO-220-3_Vertical -> Package_TO_SOT_SMD:TO-263-5_TabPin3
- Y1: value 16MHz -> 20MHz; footprint Crystal:Crystal_SMD_5032-2Pin_5.0x3.2mm -> Crystal:Crystal_HC49-4H_Vertical
- Y2: value Crystal -> 16MHz; footprint Crystal:Crystal_SMD_5032-2Pin_5.0x3.2mm -> Crystal:Crystal_HC49-4H_Vertical; moved to F.Cu
- moved D2 77.8 mm to (149.5, 100.5), turned to 180 degrees
- moved C3 76.9 mm to (113.5, 111.0)
- moved Q5 76.3 mm to (124.0, 34.0), turned to 180 degrees
- moved C12 75.1 mm to (93.3, 104.2), turned to 90 degrees
- moved R17 72.7 mm to (149.5, 100.5)
- moved R10 67.4 mm to (121.5, 43.2), turned to 90 degrees
- moved Q9 65.3 mm to (110.0, 34.0), turned to 180 degrees
- moved Q4 62.2 mm to (123.9, 48.2)
- moved R9 58.9 mm to (100.5, 43.2), turned to -90 degrees
- moved Q2 58.6 mm to (103.0, 34.0), turned to 180 degrees
- moved R6 55.1 mm to (89.5, 74.0)
- moved Q10 54.6 mm to (103.1, 48.2)
- moved R14 54.3 mm to (107.5, 43.2), turned to -90 degrees
- moved Q7 54.1 mm to (117.0, 34.0), turned to 180 degrees
- moved Q3 48.9 mm to (88.5, 79.5), turned to 90 degrees
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Connections:
- net PC3 renamed HESD_5V
- net PC4 renamed IMMOBI_5V
- C1 pad 1: +5V -> Net-(U1-AVCC)
- C12 pad 1: Net-(D1-K) -> +12V
- C2 pad 1: +5V -> Net-(U2-FB)
- C3 pad 1: Net-(D1-K) -> +12V
- C4 pad 1: +5V -> Net-(U2-FB)
- D1 pad 2: IGN -> GND
- D2 pad 1: GND -> Net-(D2-K)
- D2 pad 2: Net-(D2-A) -> +5V
- J2 pad 17: FUEL -> TEMP
- R17 pad 1: +5V -> GND
- R17 pad 2: Net-(D2-A) -> Net-(D2-K)
- U1 pad 12: CS -> Net-(U1-PB0)
- U1 pad 18: +5V -> Net-(U1-AVCC)
- U1 pad 4: +5V -> Net-(U1-AVCC)
- U1 pad 6: +5V -> Net-(U1-AVCC)
- U2 pad 1: Net-(D1-K) -> +12V
- U2 pad 2: GND -> Net-(D1-K)
- U2 pad 3: +5V -> GND
- U6 pad 7: FUEL -> TEMP
Routing:
- net FI IND: track 87.5 -> 0.00 mm, vias 1 -> 0
- net FUEL: track 83.7 -> 0.00 mm, vias 9 -> 0
- net GND: track 71.2 -> 0.00 mm, vias 3 -> 0
- net +12V: track 95.0 -> 29.6 mm, vias 5 -> 0
- net +5V: track 57.9 -> 2.95 mm, vias 3 -> 0
- net MOSI: track 52.2 -> 0.03 mm, vias 2 -> 0
- net TACHO: track 20.8 -> 69.5 mm
- net PD4: track 3.32 -> 44.2 mm
- net CANH: track 42.2 -> 4.84 mm
- net IGN: track 35.3 -> 0.00 mm
- net Net-(U2-FB): track 0.00 -> 34.2 mm
- net CS1: track 5.41 -> 38.3 mm
- net MISO: track 32.6 -> 0.00 mm, vias 3 -> 0
- net Net-(U1-PC0): track 38.2 -> 6.16 mm, vias 2 -> 1
- net SCK: track 32.0 -> 0.00 mm, vias 2 -> 0
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- added copper zone on F.Cu, net GND
